File: Triple Half Bridge Driver v3/PCB/PCB.kicad_pcb (KiCad board)
At the start: 2 copper layers, 220 x 160 mm, 119 parts, among them J1 Screw_Terminal_01x06, J10 Screw_Terminal_01x03, J11 Screw_Terminal_01x03, J12 Screw_Terminal_01x03, J13 Screw_Terminal_01x02, J2 Screw_Terminal_01x03, J3 Screw_Terminal_01x03, J4 Screw_Terminal_01x03, J5 Screw_Terminal_01x03, J6 Screw_Terminal_01x02, J7 Screw_Terminal_01x03, J8 Screw_Terminal_01x03, J9 Screw_Terminal_01x03, Q1 IRF740, Q10 IRF740, Q11 IRF740, Q12 IRF740, Q2 IRF740, Q3 IRF740, Q4 IRF740, Q5 IRF740, Q6 IRF740, Q7 IRF740, Q8 IRF740, Q9 IRF740, U1 IRS2104, U2 IRS2104, U3 IRS2104, U4 RaspberryPi_Pico, U5 IRS2104, U6 IRS2104, U7 IRS2104, U8 LM393, U9 LM393

Commit message: Add tracks for PCB
Parts:
- removed Q11, Q12: IRF740, Package_TO_SOT_THT:TO-220-3_Vertical
- removed TP31, TP32, TP33, TP34, TP35, TP36, TP37: TestPoint, TestPoint:TestPoint_THTPad_2.0x2.0mm_Drill1.0mm
- added C11: 4.7uF 35V, Capacitor_THT:C_Rect_L7.0mm_W4.5mm_P5.00mm, F.Cu at (300.0, 55.0)
- added C12: C, Capacitor_THT:C_Rect_L7.0mm_W4.5mm_P5.00mm, F.Cu at (354.5, 67.5)
- added C13: C, Capacitor_THT:C_Rect_L7.0mm_W4.5mm_P5.00mm, F.Cu at (354.0, 56.0)
- added C14: C, Capacitor_THT:C_Rect_L7.0mm_W4.5mm_P5.00mm, F.Cu at (354.5, 73.5)
- added C15: C, Capacitor_THT:C_Rect_L7.0mm_W4.5mm_P5.00mm, F.Cu at (320.0, 59.5)
- added C16: 4.7uF 35V, Capacitor_THT:C_Rect_L7.0mm_W4.5mm_P5.00mm, F.Cu at (303.0, 90.3)
- added C17: C, Capacitor_THT:C_Rect_L7.0mm_W4.5mm_P5.00mm, F.Cu at (321.5, 96.3)
- added C18: C, Capacitor_THT:C_Rect_L7.0mm_W4.5mm_P5.00mm, F.Cu at (355.6, 106.5)
- added C19: C, Capacitor_THT:C_Rect_L7.0mm_W4.5mm_P5.00mm, F.Cu at (355.6, 96.0)
- added C20: C, Capacitor_THT:C_Rect_L7.0mm_W4.5mm_P5.00mm, F.Cu at (355.6, 113.0)
- added C21: 4.7uF 35V, Capacitor_THT:C_Rect_L7.0mm_W4.5mm_P5.00mm, F.Cu at (302.5, 128.8)
- added C22: C, Capacitor_THT:C_Rect_L7.0mm_W4.5mm_P5.00mm, F.Cu at (321.0, 135.8)
- added C23: C, Capacitor_THT:C_Rect_L7.0mm_W4.5mm_P5.00mm, F.Cu at (360.5, 143.4)
- added C24: C, Capacitor_THT:C_Rect_L7.0mm_W4.5mm_P5.00mm, F.Cu at (355.5, 131.9)
- added C25: C, Capacitor_THT:C_Rect_L7.0mm_W4.5mm_P5.00mm, F.Cu at (355.5, 150.4)
- added C26: C, Capacitor_THT:C_Rect_L7.0mm_W4.5mm_P5.00mm, F.Cu at (238.6, 121.7)
- added C27: C, Capacitor_THT:C_Rect_L7.0mm_W4.5mm_P5.00mm, F.Cu at (239.0, 140.5)
- added C28: C, Capacitor_THT:C_Rect_L7.0mm_W4.5mm_P5.00mm, F.Cu at (244.0, 159.5)
- added C29: C, Capacitor_THT:C_Rect_L7.0mm_W4.5mm_P5.00mm, F.Cu at (238.1, 60.5)
- added C30: C, Capacitor_THT:C_Rect_L7.0mm_W4.5mm_P5.00mm, F.Cu at (243.6, 79.0)
- added C31: C, Capacitor_THT:C_Rect_L7.0mm_W4.5mm_P5.00mm, F.Cu at (285.5, 180.2)
- added C32: C, Capacitor_THT:C_Rect_L7.0mm_W4.5mm_P5.00mm, F.Cu at (299.5, 180.2)
- added C33: C, Capacitor_THT:C_Rect_L7.0mm_W4.5mm_P5.00mm, F.Cu at (257.5, 181.2)
- added C34: C, Capacitor_THT:C_Rect_L7.0mm_W4.5mm_P5.00mm, F.Cu at (271.5, 181.2)
- added C35: C, Capacitor_THT:C_Rect_L7.0mm_W4.5mm_P5.00mm, F.Cu at (161.0, 174.4)
- added C36: C, Capacitor_THT:C_Rect_L7.0mm_W4.5mm_P5.00mm, F.Cu at (62.9, 194.8)
- added C37: C, Capacitor_THT:C_Rect_L7.0mm_W4.5mm_P5.00mm, F.Cu at (47.9, 195.8)
- added C38: C, Capacitor_THT:C_Rect_L7.0mm_W4.5mm_P5.00mm, F.Cu at (53.9, 226.9)
- added C39: C, Capacitor_THT:C_Rect_L7.0mm_W4.5mm_P5.00mm, F.Cu at (63.4, 226.9)
- added C40: C, Capacitor_THT:C_Rect_L7.0mm_W4.5mm_P5.00mm, F.Cu at (55.1, 261.6)
- added C41: C, Capacitor_THT:C_Rect_L7.0mm_W4.5mm_P5.00mm, F.Cu at (64.1, 241.1)
- added C42: C, Capacitor_THT:C_Rect_L7.0mm_W4.5mm_P5.00mm, F.Cu at (116.3, 258.2)
- added C43: C, Capacitor_THT:C_Rect_L7.0mm_W4.5mm_P5.00mm, F.Cu at (124.3, 238.7)
- added C44: C, Capacitor_THT:C_Rect_L7.0mm_W4.5mm_P5.00mm, F.Cu at (115.0, 230.0)
- added C45: C, Capacitor_THT:C_Rect_L7.0mm_W4.5mm_P5.00mm, F.Cu at (121.5, 210.5)
- added C46: C, Capacitor_THT:C_Rect_L7.0mm_W4.5mm_P5.00mm, F.Cu at (115.2, 201.3)
- added C47: C, Capacitor_THT:C_Rect_L7.0mm_W4.5mm_P5.00mm, F.Cu at (120.7, 182.8)
- added C48: C, Capacitor_THT:C_Rect_L7.0mm_W4.5mm_P5.00mm, F.Cu at (359.0, 49.0)
- added C49: C, Capacitor_THT:C_Rect_L7.0mm_W4.5mm_P5.00mm, F.Cu at (360.6, 89.5)
- added C50: C, Capacitor_THT:C_Rect_L7.0mm_W4.5mm_P5.00mm, F.Cu at (360.5, 125.4)
- added C51: C, Capacitor_THT:C_Rect_L7.0mm_W4.5mm_P5.00mm, F.Cu at (243.1, 53.5)
- added C52: C, Capacitor_THT:C_Rect_L7.0mm_W4.5mm_P5.00mm, F.Cu at (243.6, 97.2)
- added C53: C, Capacitor_THT:C_Rect_L7.0mm_W4.5mm_P5.00mm, F.Cu at (244.0, 133.5)
- added C54: C, Capacitor_THT:C_Rect_L7.0mm_W4.5mm_P5.00mm, F.Cu at (55.4, 177.3)
- added C55: C, Capacitor_THT:C_Rect_L7.0mm_W4.5mm_P5.00mm, F.Cu at (59.4, 207.4)
- added C56: C, Capacitor_THT:C_Rect_L7.0mm_W4.5mm_P5.00mm, F.Cu at (64.1, 261.6)
- added C57: C, Capacitor_THT:C_Rect_L7.0mm_W4.5mm_P5.00mm, F.Cu at (124.7, 201.3)
- added C58: C, Capacitor_THT:C_Rect_L7.0mm_W4.5mm_P5.00mm, F.Cu at (125.5, 230.0)
- added C59: C, Capacitor_THT:C_Rect_L7.0mm_W4.5mm_P5.00mm, F.Cu at (126.8, 258.2)
- added D10: D, Diode_THT:D_A-405_P7.62mm_Horizontal, F.Cu at (315.3, 90.3)
- added D11: D_Schottky, Diode_THT:D_A-405_P7.62mm_Horizontal, F.Cu at (333.7, 91.3)
- added D12: D_Schottky, Diode_THT:D_A-405_P7.62mm_Horizontal, F.Cu at (334.2, 105.8)
- added D13: D, Diode_THT:D_A-405_P7.62mm_Horizontal, F.Cu at (314.3, 129.8)
- added D14: D_Schottky, Diode_THT:D_A-405_P7.62mm_Horizontal, F.Cu at (333.5, 131.3)
- added D15: D_Schottky, Diode_THT:D_A-405_P7.62mm_Horizontal, F.Cu at (333.7, 147.8)
- added D16: D_Schottky, Diode_THT:D_A-405_P7.62mm_Horizontal, F.Cu at (215.3, 118.2)
- added D17: D_Schottky, Diode_THT:D_A-405_P7.62mm_Horizontal, F.Cu at (216.9, 152.5)
- added D18: D_Schottky, Diode_THT:D_A-405_P7.62mm_Horizontal, F.Cu at (214.8, 74.0)
- added D25: D_Schottky, Diode_THT:D_A-405_P7.62mm_Horizontal, F.Cu at (174.5, 170.7)
- added D26: LED, LED_THT:LED_D5.0mm, F.Cu at (52.1, 149.4)
- added D27: LED, LED_THT:LED_D5.0mm, F.Cu at (51.8, 159.4)
- added D7: D, Diode_THT:D_A-405_P7.62mm_Horizontal, F.Cu at (313.8, 53.5)
- added D8: D_Schottky, Diode_THT:D_A-405_P7.62mm_Horizontal, F.Cu at (331.7, 56.0)
- added D9: D_Schottky, Diode_THT:D_A-405_P7.62mm_Horizontal, F.Cu at (332.2, 73.0)
- added FB1: FerriteBead, Ferrite_THT:LairdTech_28C0236-0JW-10, F.Cu at (140.0, 104.0)
- added FB2: FerriteBead, Ferrite_THT:LairdTech_28C0236-0JW-10, F.Cu at (174.0, 176.9)
- added J14: Screw_Terminal_01x03, 3 Pin Spring Terminal:1792876, F.Cu at (373.0, 97.5)
- added J15: Screw_Terminal_01x03, Connector_PinHeader_2.54mm:PinHeader_1x03_P2.54mm_Vertical, F.Cu at (56.5, 116.6)
- added J16: Screw_Terminal_01x03, Connector_PinHeader_2.54mm:PinHeader_1x03_P2.54mm_Vertical, F.Cu at (57.0, 129.6)
- added J17: Screw_Terminal_01x02, 3 Pin Spring Terminal:1792863, F.Cu at (278.0, 141.0)
- added J18: Screw_Terminal_01x02, 3 Pin Spring Terminal:1792863, F.Cu at (158.4, 69.2)
- added J19: Screw_Terminal_01x02, 3 Pin Spring Terminal:1792863, F.Cu at (158.6, 103.5)
- added J20: Screw_Terminal_01x02, 3 Pin Spring Terminal:1792863, F.Cu at (161.6, 147.0)
- added J21: Screw_Terminal_01x03, 3 Pin Spring Terminal:1792876, F.Cu at (34.0, 224.5)
- added J22: Screw_Terminal_01x03, 3 Pin Spring Terminal:1792876, F.Cu at (89.7, 214.5)
- added JP1: SolderJumper_2_Bridged, Jumper:SolderJumper-2_P1.3mm_Bridged_Pad1.0x1.5mm, F.Cu at (57.2, 195.3)
- added JP2: SolderJumper_2_Bridged, Jumper:SolderJumper-2_P1.3mm_Bridged_Pad1.0x1.5mm, F.Cu at (59.0, 226.9)
- added JP7: SolderJumper_2_Open, Jumper:SolderJumper-2_P1.3mm_Open_Pad1.0x1.5mm, F.Cu at (172.2, 182.9)
- added JP8: SolderJumper_2_Open, Jumper:SolderJumper-2_P1.3mm_Open_Pad1.0x1.5mm, F.Cu at (165.3, 182.9)
- added Q13: Q_PNP_BEC, Package_TO_SOT_THT:TO-220-3_Vertical, F.Cu at (314.0, 80.5)
- added Q14: IRF740, Package_TO_SOT_THT:TO-220-3_Vertical, F.Cu at (347.0, 55.5)
- added Q15: IRF740, Package_TO_SOT_THT:TO-220-3_Vertical, F.Cu at (347.0, 67.5)
- added Q16: Q_PNP_BEC, Package_TO_SOT_THT:TO-220-3_Vertical, F.Cu at (315.0, 117.3)
- added Q17: IRF740, Package_TO_SOT_THT:TO-220-3_Vertical, F.Cu at (349.1, 92.4)
- added Q18: IRF740, Package_TO_SOT_THT:TO-220-3_Vertical, F.Cu at (348.6, 104.9)
- added Q19: Q_PNP_BEC, Package_TO_SOT_THT:TO-220-3_Vertical, F.Cu at (314.4, 154.8)
- added Q20: IRF740, Package_TO_SOT_THT:TO-220-3_Vertical, F.Cu at (346.5, 131.4)
- added Q21: IRF740, Package_TO_SOT_THT:TO-220-3_Vertical, F.Cu at (346.5, 144.4)
- added R29: R, Resistor_THT:R_Axial_DIN0207_L6.3mm_D2.5mm_P7.62mm_Horizontal, F.Cu at (331.7, 62.0)
- added R30: R, Resistor_THT:R_Axial_DIN0207_L6.3mm_D2.5mm_P7.62mm_Horizontal, F.Cu at (331.9, 67.5)
- added R31: R, Resistor_THT:R_Axial_DIN0207_L6.3mm_D2.5mm_P7.62mm_Horizontal, F.Cu at (288.5, 54.1)
- added R32: R, Resistor_THT:R_Axial_DIN0207_L6.3mm_D2.5mm_P7.62mm_Horizontal, F.Cu at (289.0, 68.7)
- added R33: R, Resistor_THT:R_Axial_DIN0207_L6.3mm_D2.5mm_P7.62mm_Horizontal, F.Cu at (320.1, 74.2)
- added R34: R, Resistor_THT:R_Axial_DIN0207_L6.3mm_D2.5mm_P7.62mm_Horizontal, F.Cu at (332.2, 78.5)
- added R35: R, Resistor_THT:R_Axial_DIN0207_L6.3mm_D2.5mm_P7.62mm_Horizontal, F.Cu at (361.3, 62.0)
- added R36: R, Resistor_THT:R_Axial_DIN0207_L6.3mm_D2.5mm_P7.62mm_Horizontal, F.Cu at (346.9, 79.0)
- added R37: R, Resistor_THT:R_Axial_DIN0207_L6.3mm_D2.5mm_P7.62mm_Horizontal, F.Cu at (291.0, 89.5)
- added R38: R, Resistor_THT:R_Axial_DIN0207_L6.3mm_D2.5mm_P7.62mm_Horizontal, F.Cu at (291.0, 103.3)
- added R39: R, Resistor_THT:R_Axial_DIN0207_L6.3mm_D2.5mm_P7.62mm_Horizontal, F.Cu at (321.0, 110.5)
- added R40: R, Resistor_THT:R_Axial_DIN0207_L6.3mm_D2.5mm_P7.62mm_Horizontal, F.Cu at (333.7, 100.8)
- added R41: R, Resistor_THT:R_Axial_DIN0207_L6.3mm_D2.5mm_P7.62mm_Horizontal, F.Cu at (333.7, 96.3)
- added R42: R, Resistor_THT:R_Axial_DIN0207_L6.3mm_D2.5mm_P7.62mm_Horizontal, F.Cu at (333.7, 111.3)
- added R43: R, Resistor_THT:R_Axial_DIN0207_L6.3mm_D2.5mm_P7.62mm_Horizontal, F.Cu at (362.1, 101.0)
- added R44: R, Resistor_THT:R_Axial_DIN0207_L6.3mm_D2.5mm_P7.62mm_Horizontal, F.Cu at (347.8, 118.0)
- added R45: R, Resistor_THT:R_Axial_DIN0207_L6.3mm_D2.5mm_P7.62mm_Horizontal, F.Cu at (289.5, 127.5)
- added R46: R, Resistor_THT:R_Axial_DIN0207_L6.3mm_D2.5mm_P7.62mm_Horizontal, F.Cu at (289.5, 141.3)
- added R47: R, Resistor_THT:R_Axial_DIN0207_L6.3mm_D2.5mm_P7.62mm_Horizontal, F.Cu at (321.0, 148.5)
- added R48: R, Resistor_THT:R_Axial_DIN0207_L6.3mm_D2.5mm_P7.62mm_Horizontal, F.Cu at (333.2, 141.8)
- added R49: R, Resistor_THT:R_Axial_DIN0207_L6.3mm_D2.5mm_P7.62mm_Horizontal, F.Cu at (333.4, 136.3)
- added R50: R, Resistor_THT:R_Axial_DIN0207_L6.3mm_D2.5mm_P7.62mm_Horizontal, F.Cu at (333.0, 153.3)
- added R51: R, Resistor_THT:R_Axial_DIN0207_L6.3mm_D2.5mm_P7.62mm_Horizontal, F.Cu at (361.8, 137.4)
- added R52: R, Resistor_THT:R_Axial_DIN0207_L6.3mm_D2.5mm_P7.62mm_Horizontal, F.Cu at (349.9, 156.9)
- added R53: R, Resistor_THT:R_Axial_DIN0207_L6.3mm_D2.5mm_P7.62mm_Horizontal, F.Cu at (215.0, 96.2)
- added R54: R, Resistor_THT:R_Axial_DIN0207_L6.3mm_D2.5mm_P7.62mm_Horizontal, F.Cu at (216.7, 136.0)
- added R55: R, Resistor_THT:R_Axial_DIN0207_L6.3mm_D2.5mm_P7.62mm_Horizontal, F.Cu at (214.3, 56.5)
- added R56: R, Resistor_THT:R_Axial_DIN0207_L6.3mm_D2.5mm_P7.62mm_Horizontal, F.Cu at (215.3, 112.7)
- added R57: R, Resistor_THT:R_Axial_DIN0207_L6.3mm_D2.5mm_P7.62mm_Horizontal, F.Cu at (216.9, 157.5)
- added R58: R, Resistor_THT:R_Axial_DIN0207_L6.3mm_D2.5mm_P7.62mm_Horizontal, F.Cu at (214.3, 80.0)
- added R59: R, Resistor_THT:R_Axial_DIN0207_L6.3mm_D2.5mm_P7.62mm_Horizontal, F.Cu at (245.1, 109.7)
- added R60: R, Resistor_THT:R_Axial_DIN0207_L6.3mm_D2.5mm_P7.62mm_Horizontal, F.Cu at (226.8, 125.2)
- added R61: R, Resistor_THT:R_Axial_DIN0207_L6.3mm_D2.5mm_P7.62mm_Horizontal, F.Cu at (245.8, 146.5)
- added R62: R, Resistor_THT:R_Axial_DIN0207_L6.3mm_D2.5mm_P7.62mm_Horizontal, F.Cu at (227.2, 162.0)
- added R63: R, Resistor_THT:R_Axial_DIN0207_L6.3mm_D2.5mm_P7.62mm_Horizontal, F.Cu at (244.8, 66.0)
- added R64: R, Resistor_THT:R_Axial_DIN0207_L6.3mm_D2.5mm_P7.62mm_Horizontal, F.Cu at (227.5, 83.0)
- added R65: R, Resistor_THT:R_Axial_DIN0207_L6.3mm_D2.5mm_P7.62mm_Horizontal, F.Cu at (102.1, 252.2)
- added R66: R, Resistor_THT:R_Axial_DIN0207_L6.3mm_D2.5mm_P7.62mm_Horizontal, F.Cu at (113.8, 244.7)
- added R67: R, Resistor_THT:R_Axial_DIN0207_L6.3mm_D2.5mm_P7.62mm_Horizontal, F.Cu at (118.3, 244.4)
- added R68: R, Resistor_THT:R_Axial_DIN0207_L6.3mm_D2.5mm_P7.62mm_Horizontal, F.Cu at (99.5, 224.0)
- added R69: R, Resistor_THT:R_Axial_DIN0207_L6.3mm_D2.5mm_P7.62mm_Horizontal, F.Cu at (116.0, 216.7)
- added R70: R, Resistor_THT:R_Axial_DIN0207_L6.3mm_D2.5mm_P7.62mm_Horizontal, F.Cu at (111.5, 216.5)
- added R71: R, Resistor_THT:R_Axial_DIN0207_L6.3mm_D2.5mm_P7.62mm_Horizontal, F.Cu at (99.6, 195.3)
- added R72: R, Resistor_THT:R_Axial_DIN0207_L6.3mm_D2.5mm_P7.62mm_Horizontal, F.Cu at (116.7, 188.0)
- added R73: R, Resistor_THT:R_Axial_DIN0207_L6.3mm_D2.5mm_P7.62mm_Horizontal, F.Cu at (111.7, 188.0)
- added R74: R, Resistor_THT:R_Axial_DIN0207_L6.3mm_D2.5mm_P7.62mm_Horizontal, F.Cu at (59.3, 149.4)
- added R75: R, Resistor_THT:R_Axial_DIN0207_L6.3mm_D2.5mm_P7.62mm_Horizontal, F.Cu at (59.3, 158.9)
- added R76: R, Resistor_THT:R_Axial_DIN0207_L6.3mm_D2.5mm_P7.62mm_Horizontal, F.Cu at (82.4, 158.9)
- added R77: 0, Resistor_THT:R_Axial_DIN0207_L6.3mm_D2.5mm_P7.62mm_Horizontal, F.Cu at (134.2, 112.0)
- added RV1: R_Potentiometer, Potentiometer_THT:Potentiometer_Omeg_PC16BU_Vertical, F.Cu at (107.6, 160.3)
- added SW1: SW_Push, Button_Switch_THT:SW_PUSH_6mm_H8.5mm, F.Cu at (75.4, 149.1)
- added TP38: TestPoint, TestPoint:TestPoint_THTPad_2.0x2.0mm_Drill1.0mm, F.Cu at (296.0, 62.5)
- added TP39: TestPoint, TestPoint:TestPoint_THTPad_2.0x2.0mm_Drill1.0mm, F.Cu at (296.0, 68.0)
- added TP40: TestPoint, TestPoint:TestPoint_THTPad_2.0x2.0mm_Drill1.0mm, F.Cu at (326.0, 56.0)
- added TP41: TestPoint, TestPoint:TestPoint_THTPad_2.0x2.0mm_Drill1.0mm, F.Cu at (327.0, 73.5)
- added TP42: TestPoint, TestPoint:TestPoint_THTPad_2.0x2.0mm_Drill1.0mm, F.Cu at (298.0, 97.8)
- added TP43: TestPoint, TestPoint:TestPoint_THTPad_2.0x2.0mm_Drill1.0mm, F.Cu at (298.0, 104.3)
- added TP44: TestPoint, TestPoint:TestPoint_THTPad_2.0x2.0mm_Drill1.0mm, F.Cu at (327.5, 91.8)
- added TP45: TestPoint, TestPoint:TestPoint_THTPad_2.0x2.0mm_Drill1.0mm, F.Cu at (328.0, 108.8)
- added TP46: TestPoint, TestPoint:TestPoint_THTPad_2.0x2.0mm_Drill1.0mm, F.Cu at (296.5, 135.3)
- added TP47: TestPoint, TestPoint:TestPoint_THTPad_2.0x2.0mm_Drill1.0mm, F.Cu at (296.5, 142.3)
- added TP48: TestPoint, TestPoint:TestPoint_THTPad_2.0x2.0mm_Drill1.0mm, F.Cu at (328.0, 131.3)
- added TP49: TestPoint, TestPoint:TestPoint_THTPad_2.0x2.0mm_Drill1.0mm, F.Cu at (327.1, 147.8)
- added U10: IRS2101, Package_DIP:DIP-8_W7.62mm, F.Cu at (308.2, 97.0)
- added U11: IRS2101, Package_DIP:DIP-8_W7.62mm, F.Cu at (306.2, 59.7)
- added U12: IRS2101, Package_DIP:DIP-8_W7.62mm, F.Cu at (307.2, 134.5)
- added U13: INA240A1D, Package_DIP:DIP-8_W7.62mm, F.Cu at (124.2, 252.3)
- added U14: INA240A1D, Package_DIP:DIP-8_W7.62mm, F.Cu at (121.7, 224.3)
- added U15: INA240A1D, Package_DIP:DIP-8_W7.62mm, F.Cu at (122.4, 195.6)
- C1, C2, C3: value 10uF -> 4.7uF 35V
- C10, C4, C5, C6, C7, C8, C9: value 10uF -> C
- D4, D5, D6: value D -> D_Schottky
- J10, J11, J12, J9: value Screw_Terminal_01x03 -> Screw_Terminal_01x02; footprint Connector_PinHeader_2.54mm:PinHeader_1x03_P2.54mm_Vertical -> 3 Pin Spring Terminal:1792863
- J13: value Screw_Terminal_01x02 -> Screw_Terminal_01x03; footprint Connector_PinSocket_2.54mm:PinSocket_1x02_P2.54mm_Vertical -> Connector_PinHeader_2.54mm:PinHeader_1x03_P2.54mm_Vertical
- J5: footprint 3 Pin Spring Terminal:1792876 -> Connector_PinHeader_2.54mm:PinHeader_1x03_P2.54mm_Vertical
- J7, J8: value Screw_Terminal_01x03 -> Screw_Terminal_01x06; footprint Connector_PinHeader_2.54mm:PinHeader_1x03_P2.54mm_Vertical -> Connector_PinHeader_2.54mm:PinHeader_1x06_P2.54mm_Vertical
- JP3, JP4, JP5: value SolderJumper_3_Bridged12 -> SolderJumper_2_Bridged; footprint Jumper:SolderJumper-3_P2.0mm_Open_TrianglePad1.0x1.5mm -> Jumper:SolderJumper-2_P1.3mm_Bridged_Pad1.0x1.5mm
- JP6: value SolderJumper_3_Open -> SolderJumper_2_Bridged; footprint Jumper:SolderJumper-3_P1.3mm_Open_Pad1.0x1.5mm -> Jumper:SolderJumper-2_P1.3mm_Bridged_Pad1.0x1.5mm
- Q1, Q2, Q3: value IRF740 -> Q_PNP_BEC
- Q10: value IRF740 -> IRF9540N
- R1, R10, R11, R12, R2, R3, R4, R5, R6, R7, R8, R9: value 10 -> R
- R13, R14, R15, R16, R17, R18: value 33k -> 10k
- R19, R20, R21: value 4.6k -> R
- R22, R23, R24, R25, R26, R27, R28: value 10k -> R
- U1, U2, U3: value IRS2104 -> IRS2101
- U4: footprint Raspberry Pi Pico:RaspberryPi_Pico_Common_THT -> Module_RaspberryPi_Pico:RaspberryPi_Pico_Common_THT
- U5: value IRS2104 -> LM7812_TO220; footprint Package_DIP:DIP-8_W7.62mm -> Package_TO_SOT_THT:TO-220-3_Vertical
- U6: value IRS2104 -> LM7805_TO220; footprint Package_DIP:DIP-8_W7.62mm -> Package_TO_SOT_THT:TO-220-3_Vertical
- U7: value IRS2104 -> INA240A1D
- U8, U9: value LM393 -> INA240A1D
- moved JP3 256.7 mm to (59.6, 261.6), turned to 0 degrees
- moved J5 245.2 mm to (56.5, 91.5), turned to 90 degrees
- moved JP4 214.4 mm to (121.3, 257.2)
- moved JP5 206.9 mm to (120.8, 230.5)
- moved TP23 182.5 mm to (73.1, 261.1)
- moved J3 177.7 mm to (57.0, 65.6), turned to 90 degrees
- moved U7 171.0 mm to (67.1, 189.6), turned to 90 degrees
- moved R26 169.8 mm to (42.9, 254.6), turned to 0 degrees
- moved TP28 168.4 mm to (131.8, 240.2)
- moved TP24 165.2 mm to (72.1, 242.1)
- moved TP21 163.2 mm to (73.4, 226.4)
- moved J9 160.9 mm to (158.5, 238.5), turned to 180 degrees
- moved TP13 160.9 mm to (67.5, 63.6)
- moved R23 160.5 mm to (43.5, 220.9), turned to 0 degrees
- moved R13 159.7 mm to (55.4, 59.9)
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Connections:
- C1 pad 1: GND -> +12V
- C1 pad 2: +3V3 -> GND
- C10 pad 2: GND -> Net-(C10-Pad2)
- C2 pad 1: Net-(D1-K) -> +12V
- C2 pad 2: Load 2A -> GND
- C3 pad 1: Net-(D4-K) -> +12V
- C3 pad 2: Load 1A -> GND
- C4 pad 1: Net-(D5-K) -> Net-(D1-K)
- C4 pad 2: Load 1B -> Motor 2B
- C5 pad 2: Load 2B -> Motor 2C
- C6 pad 1: Net-(D6-K) -> Net-(D3-K)
- C6 pad 2: Load 1C -> Motor 2A
- C7 pad 1: GND -> Low 2B2
- C7 pad 2: +3V3 -> GND
- C8 pad 1: Net-(D3-K) -> Low 2C2
- C8 pad 2: Load 2C -> GND
- C9 pad 1: VPP -> Low 2A2
- D1 pad 2: +3V3 -> +12V
- D2 pad 2: +3V3 -> +12V
- D3 pad 2: +3V3 -> +12V
- D4 pad 1: Net-(D4-K) -> High 2B1
- D4 pad 2: +3V3 -> High 2B2
- D5 pad 1: Net-(D5-K) -> High 2C1
- D5 pad 2: +3V3 -> High 2C2
- D6 pad 1: Net-(D6-K) -> High 2A1
- D6 pad 2: +3V3 -> High 2A2
- J10 pad 1: +5V -> GND1
- J10 pad 2: GND -> Reference Voltage
- J11 pad 1: +5V -> Gate 1AL
- J11 pad 2: GND -> Gate 1AH
- J12 pad 1: +5V -> Gate 1BL
- J12 pad 2: GND -> Gate 1BH
- J13 pad 2: GND -> GND1
- J2 pad 1: Load 1A -> Motor 2A
- J2 pad 2: Load 1B -> Motor 2B
- J2 pad 3: Load 1C -> Motor 2C
- J3 pad 1: Gate 2A -> +5V
- J3 pad 2: Gate 2B -> GND1
- J3 pad 3: Gate 2C -> Hall 1
- J4 pad 1: Gate 1A -> +5V
- J4 pad 2: Gate 1B -> GND1
- J4 pad 3: Gate 1C -> Hall 2
- J5 pad 1: Load 2A -> +5V
- J5 pad 2: Load 2B -> GND1
- J5 pad 3: Load 2C -> Hall 3
- J6 pad 1: VPP -> VSS
- J7 pad 1: +5V -> Sensor 1A
- J7 pad 2: GND -> Sensor 1B
- J7 pad 3: Net-(J7-Pin_3) -> Sensor 1C
- J8 pad 1: +5V -> Net-(J8-Pin_1)
- J8 pad 2: GND -> Net-(J8-Pin_2)
- J9 pad 1: +5V -> Reference Voltage
- J9 pad 2: GND -> +3V3
- JP3 pad 1: Motor A -> Net-(JP3-A)
- JP3 pad 2: Load 1C -> Net-(JP3-B)
- JP4 pad 1: Motor B -> Net-(JP4-A)
- JP4 pad 2: Load 1B -> Net-(JP4-B)
- JP5 pad 1: Motor C -> Net-(JP5-A)
- JP5 pad 2: Load 1A -> Net-(JP5-B)
- JP6 pad 1: +3V3 -> Net-(JP6-A)
- JP6 pad 2: Net-(JP6-C) -> Net-(JP6-B)
- Q1 pad 1: Low 2A2 -> Net-(Q1-B)
- Q1 pad 2: Load 2A -> Net-(Q1-E)
- Q10 pad 1: Low 1B2 -> Net-(Q10-G)
- Q10 pad 2: Load 1B -> VSS
- Q10 pad 3: GND -> Net-(D25-K)
- Q2 pad 1: Low 2B2 -> Net-(Q2-B)
- Q2 pad 2: Load 2B -> Net-(Q2-E)
- Q3 pad 1: High 2B2 -> Net-(Q3-B)
- Q3 pad 2: VPP -> Net-(Q3-E)
- Q3 pad 3: Load 2B -> GND
- Q4 pad 1: High 2C2 -> High 2B2
- Q4 pad 3: Load 2C -> Motor 2B
- Q5 pad 1: Low 2C2 -> Low 2B2
- Q5 pad 2: Load 2C -> Motor 2B
- Q6 pad 1: High 1A2 -> High 2C2
- Q6 pad 3: Load 1A -> Motor 2C
- Q7 pad 1: High 2A2 -> Low 2C2
- Q7 pad 2: VPP -> Motor 2C
- Q7 pad 3: Load 2A -> GND
- Q8 pad 1: Low 1A2 -> High 2A2
- Q8 pad 2: Load 1A -> VPP
- Q8 pad 3: GND -> Motor 2A
- Q9 pad 1: High 1B2 -> Low 2A2
- Q9 pad 2: VPP -> Motor 2A
- Q9 pad 3: Load 1B -> GND
- R1 pad 1: High 2A1 -> GND
- R1 pad 2: High 2A2 -> Gate 2BH
- R10 pad 1: Low 1B1 -> Low 2B1
- R10 pad 2: Low 1B2 -> Low 2B2
- R11 pad 1: High 1C1 -> Low 2C1
- R11 pad 2: High 1C2 -> Low 2C2
- R12 pad 1: Low 1C1 -> Low 2A1
- R12 pad 2: Low 1C2 -> Low 2A2
- R13 pad 1: Net-(U8A-+) -> +5V
- R13 pad 2: Net-(U9A--) -> Hall 1
- R14 pad 1: Net-(U8A-+) -> +5V
- R14 pad 2: Net-(U9B--) -> Hall 2
- R15 pad 1: Net-(U8A-+) -> +5V
- R15 pad 2: Net-(U8A--) -> Hall 3
- R16 pad 1: Net-(U9A--) -> +5V
- R16 pad 2: Motor A -> Hall 4
- R17 pad 1: Net-(U9B--) -> +5V
- R17 pad 2: Motor B -> Hall 5
- R18 pad 1: Net-(U8A--) -> +5V
- R18 pad 2: Motor C -> Hall 6
- R19 pad 1: Net-(U9A--) -> Voltage Control
- R19 pad 2: GND -> Net-(Q10-G)
- R2 pad 1: Low 2A1 -> Gate 2BL
- R2 pad 2: Low 2A2 -> GND
- R20 pad 1: Net-(U9B--) -> Net-(U7-+)
- R20 pad 2: GND -> Net-(JP1-B)
- R21 pad 1: GND -> Net-(U7-+)
- R21 pad 2: Net-(U8A--) -> Net-(JP1-B)
- R22 pad 1: +5V -> Net-(J21-Pin_3)
- R22 pad 2: Net-(J9-Pin_3) -> Net-(JP1-B)
- R23 pad 1: +5V -> Net-(J21-Pin_2)
- R23 pad 2: Net-(J7-Pin_3) -> Net-(JP2-B)
- R24 pad 1: Net-(JP6-C) -> Net-(U8-+)
- R24 pad 2: Net-(U8A-+) -> Net-(JP2-B)
- R25 pad 1: +5V -> Net-(U8-+)
- R25 pad 2: Net-(J8-Pin_3) -> Net-(JP2-B)
- R26 pad 1: +5V -> Net-(J21-Pin_1)
- R26 pad 2: Net-(J10-Pin_3) -> Net-(JP3-B)
- R27 pad 1: +5V -> Net-(U9-+)
- R27 pad 2: Net-(J11-Pin_3) -> Net-(JP3-B)
- R28 pad 1: +5V -> Net-(U9-+)
- R28 pad 2: Net-(J12-Pin_3) -> Net-(JP3-B)
- R3 pad 1: High 2B1 -> GND
- R3 pad 2: High 2B2 -> Gate 2CH
- R4 pad 1: Low 2B1 -> Gate 2CL
- R4 pad 2: Low 2B2 -> GND
- R5 pad 1: High 2C1 -> GND
- R5 pad 2: High 2C2 -> Gate 2AH
- R6 pad 1: Low 2C1 -> Gate 2AL
- R6 pad 2: Low 2C2 -> GND
- R7 pad 1: High 1A1 -> Low 2B1
- R7 pad 2: High 1A2 -> Net-(Q1-B)
- R8 pad 1: Low 1A1 -> Low 2C1
- R8 pad 2: Low 1A2 -> Net-(Q2-B)
- R9 pad 1: High 1B1 -> Low 2A1
- R9 pad 2: High 1B2 -> Net-(Q3-B)
- TP1 pad 1: Gate 1A -> Gate 2BH
- TP10 pad 1: Load 1C -> Low 2C1
- TP11 pad 1: High 1C1 -> High 2A1
- TP12 pad 1: Low 1C1 -> Low 2A1
- TP13 pad 1: Net-(U8A-+) -> Hall 1
- TP14 pad 1: Net-(U4-GPIO14) -> Hall 2
- TP15 pad 1: Net-(U4-GPIO13) -> Hall 3
- TP16 pad 1: Net-(J10-Pin_3) -> Net-(JP1-B)
- TP17 pad 1: Net-(U4-GPIO15) -> Hall 6
- TP18 pad 1: Net-(U9A--) -> Hall 5
- TP19 pad 1: Net-(U9B--) -> Hall 4
- TP2 pad 1: Gate 1B -> Gate 2BL
- TP20 pad 1: Net-(U8A--) -> Sensor 1A
- TP21 pad 1: Net-(J9-Pin_3) -> Net-(JP2-B)
- TP22 pad 1: Net-(J7-Pin_3) -> Sensor 1B
- TP23 pad 1: Gate 2A -> Net-(JP3-B)
- TP24 pad 1: Gate 2B -> Sensor 1C
- TP25 pad 1: Gate 2C -> Net-(JP6-B)
- TP26 pad 1: High 2A1 -> Net-(JP5-B)
- TP27 pad 1: Low 2A1 -> Net-(JP4-B)
- TP28 pad 1: Load 2A -> Sensor 2A
- TP29 pad 1: Load 2B -> Sensor 2B
- TP3 pad 1: Gate 1C -> Gate 2CH
- TP30 pad 1: Load 2C -> Sensor 2C
- TP4 pad 1: High 1A1 -> Gate 2CL
- TP5 pad 1: Low 1A1 -> Gate 2AH
- TP6 pad 1: High 1B1 -> Gate 2AL
- TP7 pad 1: Low 1B1 -> High 2B1
- TP8 pad 1: Load 1A -> Low 2B1
- TP9 pad 1: Load 1B -> High 2C1
- U1 pad 1: +3V3 -> +12V
- U1 pad 2: Gate 2A -> Gate 2BH
- U1 pad 3: +3V3 -> Gate 2BL
- U1 pad 5: Low 2A1 -> Low 2B1
- U1 pad 6: Load 2A -> Motor 2B
- U1 pad 7: High 2A1 -> High 2B1
- U2 pad 1: +3V3 -> +12V
- U2 pad 2: Gate 2B -> Gate 2CH
- U2 pad 3: +3V3 -> Gate 2CL
- U2 pad 5: Low 2B1 -> Low 2C1
- U2 pad 6: Load 2B -> Motor 2C
- U2 pad 7: High 2B1 -> High 2C1
- U3 pad 1: +3V3 -> +12V
- U3 pad 2: Gate 2C -> Gate 2AH
- U3 pad 3: +3V3 -> Gate 2AL
- U3 pad 5: Low 2C1 -> Low 2A1
- U3 pad 6: Load 2C -> Motor 2A
- U3 pad 7: High 2C1 -> High 2A1
- U4 pad 10: Net-(J12-Pin_3) -> Hall 6
- U4 pad 11: unconnected-(U4-GPIO8-Pad11) -> Net-(J8-Pin_6)
- U4 pad 12: unconnected-(U4-GPIO9-Pad12) -> Net-(J8-Pin_5)
- U4 pad 13: GND -> GND1
- U4 pad 14: unconnected-(U4-GPIO10-Pad14) -> Net-(J8-Pin_4)
- U4 pad 15: unconnected-(U4-GPIO11-Pad15) -> Net-(J8-Pin_3)
- U4 pad 16: unconnected-(U4-GPIO12-Pad16) -> Net-(J8-Pin_2)
- U4 pad 17: Net-(U4-GPIO13) -> Net-(J8-Pin_1)
- U4 pad 18: GND -> GND1
- U4 pad 19: Net-(U4-GPIO14) -> LED 1
- U4 pad 2: unconnected-(U4-GPIO1-Pad2) -> Button 
- U4 pad 20: Net-(U4-GPIO15) -> LED 2
- U4 pad 23: GND -> GND1
- U4 pad 28: GND -> GND1
- U4 pad 29: unconnected-(U4-GPIO22-Pad29) -> Voltage Control
- U4 pad 3: GND -> GND1
- U4 pad 31: unconnected-(U4-GPIO26_ADC0-Pad31) -> Potentiometer
- U4 pad 38: GND -> GND1
- U4 pad 4: Net-(J9-Pin_3) -> Hall 1
- U4 pad 5: Net-(J7-Pin_3) -> Hall 2
- U4 pad 6: Net-(J8-Pin_3) -> Hall 3
- U4 pad 7: Net-(J10-Pin_3) -> Hall 4
- U4 pad 8: GND -> GND1
- U4 pad 9: Net-(J11-Pin_3) -> Hall 5
- U5 pad 1: +3V3 -> VSS
- U5 pad 2: Gate 1A -> GND
- U5 pad 3: +3V3 -> +12V
- U6 pad 1: +3V3 -> VSS
- U6 pad 2: Gate 1B -> GND
- U6 pad 3: +3V3 -> +5V
- U7 pad 1: +3V3 -> Net-(JP1-B)
- U7 pad 2: Gate 1C -> GND1
- U7 pad 3: +3V3 -> GND1
- U7 pad 4: GND -> GND1
- U7 pad 5: Low 1C1 -> Sensor 1A
- U7 pad 6: Load 1C -> +3V3
- U7 pad 7: High 1C1 -> Reference Voltage
- U7 pad 8: Net-(D6-K) -> Net-(U7-+)
- U8 pad 1: Net-(U4-GPIO13) -> Net-(JP2-B)
- U8 pad 2: Net-(U8A--) -> GND1
- U8 pad 3: Net-(U8A-+) -> GND1
- U8 pad 4: GND -> GND1
- U8 pad 5: unconnected-(U8B-+-Pad5) -> Sensor 1B
- U8 pad 6: unconnected-(U8B---Pad6) -> +3V3
- U8 pad 7: unconnected-(U8-Pad7) -> Reference Voltage
- U8 pad 8: +3V3 -> Net-(U8-+)
- U9 pad 1: Net-(U4-GPIO15) -> Net-(JP3-B)
- U9 pad 2: Net-(U9A--) -> GND1
- U9 pad 3: Net-(U8A-+) -> GND1
- U9 pad 4: GND -> GND1
- U9 pad 5: Net-(U8A-+) -> Sensor 1C
- U9 pad 6: Net-(U9B--) -> +3V3
- U9 pad 7: Net-(U4-GPIO14) -> Reference Voltage
- U9 pad 8: +3V3 -> Net-(U9-+)
Routing:
- net GND1: track 0.00 -> 666.9 mm
- net +12V: track 0.00 -> 370.7 mm
- net Reference Voltage: track 0.00 -> 264.5 mm
- net Motor B: track 237.5 -> 0.00 mm, vias 3 -> 0
- net VPP: track 234.1 -> 469.4 mm, vias 0 -> 2
- net GND: track 690.2 -> 469.5 mm
- net Motor C: track 214.4 -> 0.00 mm, vias 1 -> 0
- net Motor A: track 195.5 -> 0.00 mm, vias 1 -> 0
- net Load 2A: track 167.9 -> 0.00 mm
- net VSS: track 0.00 -> 166.1 mm
- net Load 1C: track 148.2 -> 0.00 mm, vias 1 -> 0
- net Load 2B: track 145.0 -> 0.00 mm, vias 1 -> 0
- net Load 1B: track 128.7 -> 0.00 mm
- net Load 2C: track 128.5 -> 0.00 mm
- net Load 1A: track 121.2 -> 0.00 mm
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- added copper zone on B.Cu, net GND1
- added copper zone on F.Cu, net GND1
Other:
- board size 220 x 160 mm -> 363.5 x 231 mm
