File: Triple Half Bridge Driver v3/PCB/PCB.kicad_sch (KiCad schematic)
At the start: 243 parts, among them J1 Screw_Terminal_01x06, J13 Screw_Terminal_01x03, J14 Screw_Terminal_01x03, J15 Screw_Terminal_01x03, J16 Screw_Terminal_01x03, J2 Screw_Terminal_01x03, J3 Screw_Terminal_01x03, J4 Screw_Terminal_01x03, J5 Screw_Terminal_01x03, J6 Screw_Terminal_01x02, J7 Screw_Terminal_01x06, J8 Screw_Terminal_01x06, Q1 Q_PNP_BEC, Q10 IRF740, Q13 Q_PNP_BEC, Q14 IRF740, Q15 IRF740, Q16 Q_PNP_BEC, Q17 IRF740, Q18 IRF740, Q19 Q_PNP_BEC, Q2 Q_PNP_BEC, Q20 IRF740, Q21 IRF740, Q3 Q_PNP_BEC, Q4 IRF740, Q5 IRF740, Q6 IRF740, Q7 IRF740, Q8 IRF740, Q9 IRF740, U1 IRS2101, U10 IRS2101, U11 IRS2101, U12 IRS2101, U13 INA240A1D, U14 INA240A1D, U15 INA240A1D, U2 IRS2101, U3 IRS2101, U4 RaspberryPi_Pico, U5 LM7812_TO220, U6 LM7805_TO220, U7 INA240A1D, U8 INA240A1D, U9 INA240A1D

Commit message: Add tracks for PCB
Parts:
- removed D19, D20, D21, D22, D23, D24: SMAJ51A, Diode_SMD:D_SMA, symbol Diode:SMF54A
- removed Q10: IRF740, Package_TO_SOT_THT:TO-220-3_Vertical, symbol Transistor_FET:IRF740
- added C48, C49, C50, C51, C52, C53, C54, C55, C56, C57, C58, C59: C, Capacitor_THT:C_Rect_L7.0mm_W4.5mm_P5.00mm, symbol Device:C
- added D26, D27: LED, LED_THT:LED_D5.0mm, symbol Device:LED
- added J10, J11, J12, J17, J18, J19, J20, J9: Screw_Terminal_01x02, 3 Pin Spring Terminal:1792863, symbol Connector:Screw_Terminal_01x02
- added J21, J22: Screw_Terminal_01x03, 3 Pin Spring Terminal:1792876, symbol Connector:Screw_Terminal_01x03
- added Q10: IRF9540N, Package_TO_SOT_THT:TO-220-3_Vertical, symbol Transistor_FET:IRF9540N
- added R74, R75, R76: R, Resistor_THT:R_Axial_DIN0207_L6.3mm_D2.5mm_P7.62mm_Horizontal, symbol Device:R
- added R77: 0, Resistor_THT:R_Axial_DIN0207_L6.3mm_D2.5mm_P7.62mm_Horizontal, symbol Device:R
- added RV1: R_Potentiometer, Potentiometer_THT:Potentiometer_Omeg_PC16BU_Vertical, symbol Device:R_Potentiometer
- added SW1: SW_Push, Button_Switch_THT:SW_PUSH_6mm_H8.5mm, symbol Switch:SW_Push
- C1, C11, C16, C2, C21, C3: footprint Capacitor_SMD:C_0603_1608Metric -> Capacitor_THT:C_Rect_L7.0mm_W4.5mm_P5.00mm
- C10, C12, C13, C14, C15, C17, C18, C19, C20, C22, C23, C24, C25, C26, C27, C28, C29, C30, C31, C32, C33, C34, C35, C36, C37, C38, C39, C4, C40, C41, C42, C43, C44, C45, C46, C47, C5, C6, C7, C8, C9: footprint (none) -> Capacitor_THT:C_Rect_L7.0mm_W4.5mm_P5.00mm
- D11, D12, D14, D15, D16, D17, D18, D25, D4, D5, D6, D8, D9: footprint (none) -> Diode_THT:D_A-405_P7.62mm_Horizontal
- FB1, FB2: footprint (none) -> Ferrite_THT:LairdTech_28C0236-0JW-10
- JP1, JP2, JP3, JP4, JP5, JP6: footprint (none) -> Jumper:SolderJumper-2_P1.3mm_Bridged_Pad1.0x1.5mm
- JP7, JP8: footprint (none) -> Jumper:SolderJumper-2_P1.3mm_Open_Pad1.0x1.5mm
- Q1, Q13, Q16, Q19, Q2, Q3: footprint Package_TO_SOT_SMD:SOT-23 -> Package_TO_SOT_THT:TO-220-3_Vertical
- R1, R10, R11, R12, R19, R2, R20, R21, R22, R23, R24, R25, R26, R27, R28, R29, R3, R30, R31, R32, R33, R34, R35, R36, R37, R38, R39, R4, R40, R41, R42, R43, R44, R45, R46, R47, R48, R49, R5, R50, R51, R52, R53, R54, R55, R56, R57, R58, R59, R6, R60, R61, R62, R63, R64, R65, R66, R67, R68, R69, R7, R70, R71, R72, R73, R8, R9: footprint (none) -> Resistor_THT:R_Axial_DIN0207_L6.3mm_D2.5mm_P7.62mm_Horizontal
- TP10, TP11, TP12, TP13, TP14, TP15, TP16, TP17, TP18, TP19, TP20, TP21, TP22, TP23, TP24, TP25, TP26, TP27, TP28, TP29, TP30, TP40, TP41, TP44, TP45, TP48, TP49, TP7, TP8, TP9: footprint (none) -> TestPoint:TestPoint_THTPad_2.0x2.0mm_Drill1.0mm
- U1, U10, U11, U12, U2, U3: footprint (none) -> Package_DIP:DIP-8_W7.62mm
- U13, U14, U15, U7, U8, U9: footprint Package_SO:SOIC-8_3.9x4.9mm_P1.27mm -> Package_DIP:DIP-8_W7.62mm
- U4: footprint Raspberry Pi Pico:RaspberryPi_Pico_Common_THT -> Module_RaspberryPi_Pico:RaspberryPi_Pico_Common_THT
Connections:
- net +12V: no longer C33.1, U6.1 (VI)
- net +3V3: now also J9.2 (Pin_2), R76.1, RV1.1; no longer U13.7 (REF1), U14.7 (REF1), U15.7 (REF1), U7.7 (REF1), U8.7 (REF1), U9.7 (REF1)
- net GND: now also R77.2; no longer C36.2, C37.2, C38.2, C39.2, C40.2, C41.2, C42.2, C43.2, C44.2, C45.2, C46.2, C47.2, FB1.2, J13.2 (Pin_2), J15.2 (Pin_2), J16.2 (Pin_2), J3.2 (Pin_2), J4.2 (Pin_2), J5.2 (Pin_2), U13.2 (GND), U13.3 (REF2), U13.4 (GND), U14.2 (GND), U14.3 (REF2), U14.4 (GND), U15.2 (GND), U15.3 (REF2), U15.4 (GND), U4.13 (GND), U4.18 (GND), U4.23 (GND), U4.28 (GND), U4.3 (GND), U4.38 (GND), U4.8 (GND), U7.2 (GND), U7.3 (REF2), U7.4 (GND), U8.2 (GND), U8.3 (REF2), U8.4 (GND), U9.2 (GND), U9.3 (REF2), U9.4 (GND)
- net Gate 1AH: now also J11.2 (Pin_2)
- net Gate 1AL: now also J11.1 (Pin_1)
- net Gate 1BH: now also J12.2 (Pin_2)
- net Gate 1BL: now also J12.1 (Pin_1)
- net Gate 1CH: now also J17.2 (Pin_2)
- net Gate 1CL: now also J17.1 (Pin_1)
- net Gate 2AH: now also J18.2 (Pin_2)
- net Gate 2AL: now also J18.1 (Pin_1)
- net Gate 2BH: now also J19.2 (Pin_2)
- net Gate 2BL: now also J19.1 (Pin_1)
- net Gate 2CH: now also J20.2 (Pin_2)
- net Gate 2CL: now also J20.1 (Pin_1)
- net High 1A2: now also C48.2
- net High 1B2: now also C49.2
- net High 1C2: now also C50.2
- net High 2A2: now also C51.2
- net High 2B2: now also C52.2
- net High 2C2: now also C53.2
- net Motor 1A: no longer R22.1
- net Motor 1B: no longer R23.1
- net Motor 1C: no longer R26.1
- net Motor 2A: no longer R65.1
- net Motor 2B: no longer R68.1
- net Motor 2C: no longer R71.1
- net VPP: now also C48.1, C49.1, C50.1, C51.1, C52.1, C53.1
- net VSS: now also C33.1, U6.1 (VI), Q10.2 (D)
- net Voltage Control: now also U4.29 (GPIO22)
- net at C35.2, D25.1 (K), FB2.1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: now also Q10.3 (S)
- net at JP1.2 (B), R20.2, R21.2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: now also C54.1
- net at R20.1, R21.1, U7.8 (+): now also C54.2
- net at C35.1, R19.2: now also Q10.1 (G)
- net at JP5.2 (B), R68.2, R69.2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: now also C58.1
- net at JP4.2 (B), R65.2, R66.2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: now also C59.1
- net at R66.1, R67.1, U13.8 (+): now also C59.2
- net at JP3.2 (B), R26.2, R27.2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: now also C56.1
- net at R27.1, R28.1, U9.8 (+): now also C56.2
- net LED 1: now reaches U4.19 (GPIO14)
- net LED 1: now also D26.2 (A)
- net Button : now reaches U4.2 (GPIO1)
- net Button : now also R76.2, SW1.1
- net LED 2: now reaches U4.20 (GPIO15)
- net LED 2: now also D27.2 (A)
- net Potentiometer: now reaches U4.31 (GPIO26_ADC0)
- net Potentiometer: now also RV1.2
- net at JP6.2 (B), R71.2, R72.2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: now also C57.1
- net at R24.1, R25.1, U8.8 (+): now also C55.2
- net at JP2.2 (B), R23.2, R24.2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: now also C55.1
- net at R69.1, R70.1, U14.8 (+): now also C58.2
- net at R72.1, R73.1, U15.8 (+): now also C57.2
- new net: D27.1 (K), R75.2
- new net: D26.1 (K), R74.2
- new net: J21.1 (Pin_1), R26.1
- new net: J21.2 (Pin_2), R23.1
- new net: J21.3 (Pin_3), R22.1
- new net: J22.3 (Pin_3), R65.1
- new net: J22.2 (Pin_2), R68.1
- new net: J22.1 (Pin_1), R71.1
- new net GND1: C36.2, C37.2, C38.2, C39.2, C40.2, C41.2, C42.2, C43.2, C44.2, C45.2, C46.2, C47.2, FB1.2, J10.1 (Pin_1), J13.2 (Pin_2), J15.2 (Pin_2), J16.2 (Pin_2), J3.2 (Pin_2), J4.2 (Pin_2), J5.2 (Pin_2), R74.1, R75.1, R77.1, RV1.3, SW1.2, U13.2 (GND), U13.3 (REF2), U13.4 (GND), U14.2 (GND), U14.3 (REF2), U14.4 (GND), U15.2 (GND), U15.3 (REF2), U15.4 (GND), U4.13 (GND), U4.18 (GND), U4.23 (GND), U4.28 (GND), U4.3 (GND), U4.38 (GND), U4.8 (GND), U7.2 (GND), U7.3 (REF2), U7.4 (GND), U8.2 (GND), U8.3 (REF2), U8.4 (GND), U9.2 (GND), U9.3 (REF2), U9.4 (GND)
- new net Reference Voltage: J10.2 (Pin_2), J9.1 (Pin_1), U13.7 (REF1), U14.7 (REF1), U15.7 (REF1), U7.7 (REF1), U8.7 (REF1), U9.7 (REF1)
Other:
- note added: "Buttons"
- moved on the sheet: C36, C37, C38, C39, C40, C41, C42, C43, C44, C45, C46, C47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
