File: PCB/Triple Half Bridge Driver v3/PCB/PCB.kicad_sch (KiCad schematic)
At the start: 267 parts, among them J1 Screw_Terminal_01x06, J10 Screw_Terminal_01x02, J11 Screw_Terminal_01x02, J12 Screw_Terminal_01x02, J13 Screw_Terminal_01x03, J14 Screw_Terminal_01x03, J15 Screw_Terminal_01x03, J16 Screw_Terminal_01x03, J17 Screw_Terminal_01x02, J18 Screw_Terminal_01x02, J19 Screw_Terminal_01x02, J2 Screw_Terminal_01x03, J20 Screw_Terminal_01x02, J21 Screw_Terminal_01x03, J22 Screw_Terminal_01x03, J3 Screw_Terminal_01x03, J4 Screw_Terminal_01x03, J5 Screw_Terminal_01x03, J6 Screw_Terminal_01x02, J7 Screw_Terminal_01x06, J8 Screw_Terminal_01x06, J9 Screw_Terminal_01x02, Q1 Q_PNP_BEC, Q10 IRF9540N, Q13 Q_PNP_BEC, Q14 IRF740, Q15 IRF740, Q16 Q_PNP_BEC, Q17 IRF740, Q18 IRF740, Q19 Q_PNP_BEC, Q2 Q_PNP_BEC, Q20 IRF740, Q21 IRF740, Q3 Q_PNP_BEC, Q4 IRF740, Q5 IRF740, Q6 IRF740, Q7 IRF740, Q8 IRF740, Q9 IRF740, SW1 SW_Push, U1 IRS2101, U10 IRS2101, U11 IRS2101, U12 IRS2101, U13 INA240A1D, U14 INA240A1D, U15 INA240A1D, U2 IRS2101, U3 IRS2101, U4 RaspberryPi_Pico, U5 LM7812_TO220, U6 LM7805_TO220, U7 INA240A1D, U8 INA240A1D, U9 INA240A1D

Commit message: Update PCB
Parts:
- added J23, J28: Screw_Terminal_01x01, Connector_PinHeader_2.54mm:PinHeader_1x01_P2.54mm_Vertical, symbol Connector:Screw_Terminal_01x01
- added J24, J25: Screw_Terminal_01x03, 3 Pin Spring Terminal:1792876, symbol Connector:Screw_Terminal_01x03
- added J26: Screw_Terminal_01x02, Connector_PinHeader_2.54mm:PinHeader_1x02_P2.54mm_Vertical, symbol Connector:Screw_Terminal_01x02
- added R78, R79, R80: R, Resistor_THT:R_Axial_DIN0207_L6.3mm_D2.5mm_P7.62mm_Horizontal, symbol Device:R
- added RV2, RV3: R_Potentiometer, Potentiometer_THT:Potentiometer_Omeg_PC16BU_Vertical, symbol Device:R_Potentiometer
- added SW2: SW_Push, Button_Switch_THT:SW_PUSH_6mm_H8.5mm, symbol Switch:SW_Push
- J10, J9: footprint 3 Pin Spring Terminal:1792863 -> Connector_PinHeader_2.54mm:PinHeader_1x02_P2.54mm_Vertical
Connections:
- net +3V3: now also R78.1, R79.1, RV2.1, RV3.1
- net +5V: now also J28.1 (Pin_1); no longer C34.1, U6.3 (VO)
- net GND1: now also R80.2, RV2.3, RV3.3, SW2.2
- net Motor 1A: now also J24.1 (Pin_1)
- net Motor 1B: now also J24.2 (Pin_2)
- net Motor 1C: now also J24.3 (Pin_3)
- net Motor 2A: now also J25.1 (Pin_1)
- net Motor 2B: now also J25.2 (Pin_2)
- net Motor 2C: now also J25.3 (Pin_3)
- net Reference Voltage: now also R79.2, R80.1
- net VSS: now also C35.1
- net at D25.1 (K), FB2.1, JP8.1 (A)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: no longer C35.2
- net Button 2: now reaches U4.1 (GPIO0)
- net Button 2: now also R78.2, SW2.1
- net Potentiometer 2: now reaches U4.32 (GPIO27_ADC1)
- net Potentiometer 2: now also RV2.2
- net Potentiometer 3: now reaches U4.34 (GPIO28_ADC2)
- net Potentiometer 3: now also RV3.2
- net at U4.40 (VBUS): now also J23.1 (Pin_1)
- net at Q10.1 (G), R19.2: now also C35.2; no longer C35.1
- net Button  renamed Button 1
- net Potentiometer renamed Potentiometer 1
- new net: C34.1, J26.1 (Pin_1), J26.2 (Pin_2), U6.3 (VO)
Other:
- moved on the sheet: C31, C32, C33, C34, D25, D26, D27, FB1, FB2, J10, J13, J15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

Commit message: Fix potentiometer footprint and overlapping silkscreen on PCB
Parts:
- RV1, RV2, RV3: footprint Potentiometer_THT:Potentiometer_Omeg_PC16BU_Vertical -> Potentiometer_THT:Potentiometer_Alps_RK09K_Single_Vertical
Changed lines of the file:
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@@
 			)
 		)
-		(property "Footprint" "Potentiometer_THT:Potentiometer_Omeg_PC16BU_Vertical"
+		(property "Footprint" "Potentiometer_THT:Potentiometer_Alps_RK09K_Single_Vertical"
 			(at 448.31 92.71 0)
 			(effects
@@
 			)
 		)
-		(property "Footprint" "Potentiometer_THT:Potentiometer_Omeg_PC16BU_Vertical"
+		(property "Footprint" "Potentiometer_THT:Potentiometer_Alps_RK09K_Single_Vertical"
 			(at 448.31 71.12 0)
 			(effects
@@
 			)
 		)
-		(property "Footprint" "Potentiometer_THT:Potentiometer_Omeg_PC16BU_Vertical"
+		(property "Footprint" "Potentiometer_THT:Potentiometer_Alps_RK09K_Single_Vertical"
 			(at 448.31 48.26 0)
 			(effects
