File: PCB/Triple Half Bridge Driver v4b2/PCB/PCB.kicad_pcb (KiCad board)
At the start: 2 copper layers, 311 x 216 mm, 365 parts, among them J1 Screw_Terminal_01x06, J10 Screw_Terminal_01x02, J100 Screw_Terminal_01x02, J101 Screw_Terminal_01x02, J102 Screw_Terminal_01x02, J103 Screw_Terminal_01x02, J11 Screw_Terminal_01x02, J12 Screw_Terminal_01x02, J13 Screw_Terminal_01x03, J14 Screw_Terminal_01x03, J15 Screw_Terminal_01x03, J16 Screw_Terminal_01x03, J17 Screw_Terminal_01x02, J18 Screw_Terminal_01x02, J19 Screw_Terminal_01x02, J2 Screw_Terminal_01x03, J20 Screw_Terminal_01x02, J21 Screw_Terminal_01x03, J23 Screw_Terminal_01x01, J24 Screw_Terminal_01x03, J25 Screw_Terminal_01x03, J26 Screw_Terminal_01x02, J27 Screw_Terminal_01x02, J28 Screw_Terminal_01x01, J29 Screw_Terminal_01x02, J3 Screw_Terminal_01x03, J30 Screw_Terminal_01x02, J31 Screw_Terminal_01x02, J32 Screw_Terminal_01x02, J33 Screw_Terminal_01x02, J34 Screw_Terminal_01x02, J35 Screw_Terminal_01x02, J36 Screw_Terminal_01x02, J37 Screw_Terminal_01x02, J38 Screw_Terminal_01x02, J39 Screw_Terminal_01x02, J4 Screw_Terminal_01x03, J40 Screw_Terminal_01x02, J41 Screw_Terminal_01x02, J42 Screw_Terminal_01x02, J43 Screw_Terminal_01x02, J44 Screw_Terminal_01x01, J45 Screw_Terminal_01x02, J46 Screw_Terminal_01x02, J47 Screw_Terminal_01x02, J48 Screw_Terminal_01x02, J49 Screw_Terminal_01x02, J5 Screw_Terminal_01x03, J50 Screw_Terminal_01x02, J51 Screw_Terminal_01x02, J52 Screw_Terminal_01x02, J53 Screw_Terminal_01x02, J54 Screw_Terminal_01x02, J55 Screw_Terminal_01x02, J56 Screw_Terminal_01x02, J57 Screw_Terminal_01x02, J58 Screw_Terminal_01x02, J59 Screw_Terminal_01x02, J6 Screw_Terminal_01x02, J60 Screw_Terminal_01x02, J61 Screw_Terminal_01x02, J62 Screw_Terminal_01x02, J63 Screw_Terminal_01x02, J64 Screw_Terminal_01x02, J65 Screw_Terminal_01x02, J66 Screw_Terminal_01x02, J67 Screw_Terminal_01x02, J68 Screw_Terminal_01x02, J69 Screw_Terminal_01x02, J7 Screw_Terminal_01x06, J70 Screw_Terminal_01x02, J71 Screw_Terminal_01x02, J72 Screw_Terminal_01x02, J73 Screw_Terminal_01x02, J74 Screw_Terminal_01x02, J75 Screw_Terminal_01x02, J76 Screw_Terminal_01x02, J77 Screw_Terminal_01x02, J78 Screw_Terminal_01x02, J79 Screw_Terminal_01x02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

Commit message: Update PCB
Parts:
- removed J10, J69, J70, J72, J73, J74, J75, J76, J79, J80, J81, J82, J86, J87, J88, J89, J90, J91, J92, J93, J94, J95, J96, J97: Screw_Terminal_01x02, 3 Pin Spring Terminal:1792863
- removed JP7: SolderJumper_2_Open, Jumper:SolderJumper-2_P1.3mm_Open_Pad1.0x1.5mm
- added RV10: R_Potentiometer, Potentiometer_THT:Potentiometer_Alps_RK09K_Single_Vertical, F.Cu at (86.9, 264.0)
- added RV11: R_Potentiometer, Potentiometer_THT:Potentiometer_Alps_RK09K_Single_Vertical, F.Cu at (86.9, 278.4)
- added RV12: R_Potentiometer, Potentiometer_THT:Potentiometer_Alps_RK09K_Single_Vertical, F.Cu at (86.9, 292.7)
- added RV13: R_Potentiometer, Potentiometer_THT:Potentiometer_Alps_RK09K_Single_Vertical, F.Cu at (102.3, 264.0)
- added RV14: R_Potentiometer, Potentiometer_THT:Potentiometer_Alps_RK09K_Single_Vertical, F.Cu at (102.3, 278.4)
- added RV15: R_Potentiometer, Potentiometer_THT:Potentiometer_Alps_RK09K_Single_Vertical, F.Cu at (102.3, 292.7)
- added RV4: R_Potentiometer, Potentiometer_THT:Potentiometer_Alps_RK09K_Single_Vertical, F.Cu at (56.0, 264.0)
- added RV5: R_Potentiometer, Potentiometer_THT:Potentiometer_Alps_RK09K_Single_Vertical, F.Cu at (56.0, 278.4)
- added RV6: R_Potentiometer, Potentiometer_THT:Potentiometer_Alps_RK09K_Single_Vertical, F.Cu at (56.0, 292.7)
- added RV7: R_Potentiometer, Potentiometer_THT:Potentiometer_Alps_RK09K_Single_Vertical, F.Cu at (71.5, 264.0)
- added RV8: R_Potentiometer, Potentiometer_THT:Potentiometer_Alps_RK09K_Single_Vertical, F.Cu at (71.5, 278.4)
- added RV9: R_Potentiometer, Potentiometer_THT:Potentiometer_Alps_RK09K_Single_Vertical, F.Cu at (71.5, 292.7)
Connections:
- FB3 pad 1: GND1 -> GND
Routing:
- net GND1: track 168.5 -> 0.00 mm, vias 1 -> 0
- net GND: track 24.2 -> 192.8 mm, vias 1 -> 2
- net Net-(J98-Pin_2): track 122.4 -> 108.2 mm
- net (no net): track 0.00 -> 14.3 mm
